File: ESP32-DSP-HW-KiCad/ESP32-DSP-HW-KiCad.kicad_sch (KiCad schematic)
At the start: 17 parts, among them IC1 TLV320ADC3120IRTER, J1 USB_C_Receptacle_USB2.0_14P, SW1 SW_Push, SW2 SW_Push, U1 ESP32-S3-WROOM-2, U2 AP7361C-33E

Commit message: More work
Parts:
- added C3: 1u, symbol Device:C
- added C4: 0.1u, symbol Device:C
- added C5: 10u, symbol Device:C
Connections:
- net GND: now also IC1.10 (VSS_2), IC1.20 (VSS_4), IC1.21 (VSS_5), IC1.22 (VSS_6), IC1.23 (VSS_7), IC1.24 (VSS_8), IC1.25 (VSS_9), IC1.5 (VSS_1), C3.2, C4.2, C5.2
- net at IC1.17 (AREG): now also C4.1, C5.1
- net at IC1.18 (VREF): now also C3.1
